File: Hardware/BMS/bms.kicad_pcb (KiCad board)
At the start: 4 copper layers, 179 x 70 mm, 319 parts, among them J101 Conn_02x02_Counter_Clockwise, J102 Conn_01x02, J103 Conn_02x05_Top_Bottom, J301 Conn_02x09_Counter_Clockwise, J302 Conn_02x09_Counter_Clockwise, J401 Conn_01x04_Socket, J402 USB_C_Receptacle_USB2.0_16P, J501 Conn_02x09_Counter_Clockwise, Q401 2N7002E, Q601 SQ2337ES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

Commit message: bms updates (for real this time)
Parts:
- removed JP1001, JP1201, JP1301, JP1401, JP1501, JP1601, JP1701, JP1801, JP1901, JP2001, JP201, JP2101, JP2201, JP701: SolderJumper_2_Open, Jumper:SolderJumper-2_P1.3mm_Open_TrianglePad1.0x1.5mm
- removed REF** (x3): TestPoint_Pad_D4.0mm, TestPoint:TestPoint_Pad_D4.0mm
- added TP929: TestPoint, TestPoint:TestPoint_Pad_1.0x1.0mm, F.Cu at (311.2, 54.6)
- added TP930: TestPoint, TestPoint:TestPoint_Pad_1.0x1.0mm, F.Cu at (313.3, 54.6)
- added kibuzzard-690BEEAD: G***, kibuzzard-690BEEAD, F.Cu at (178.1, 59.7)
- added kibuzzard-690BEF4B: G***, kibuzzard-690BEF4B, F.Cu at (178.1, 43.8)
- added kibuzzard-690CD8B4: G***, kibuzzard-690CD8B4, F.Cu at (210.2, 45.1)
- added kibuzzard-690CF627: G***, kibuzzard-690CF627, F.Cu at (310.2, 45.1)
- added kibuzzard-690CF62F: G***, kibuzzard-690CF62F, F.Cu at (310.1, 52.4)
- added kibuzzard-690CF63A: G***, kibuzzard-690CF63A, F.Cu at (210.1, 52.4)
- J102: footprint Connector_Molex:Molex_Nano-Fit_105313-xx02_1x02_P2.50mm_Horizontal -> Connector_Molex:Molex_Micro-Fit_3.0_43650-0200_1x02_P3.00mm_Horizontal
- TP801, TP802, TP803, TP804, TP805, TP806, TP807, TP808, TP809, TP810, TP811, TP812, TP813, TP814, TP815: footprint TestPoint:TestPoint_Pad_1.0x1.0mm -> TestPoint:TestPoint_Keystone_5019_Miniature
- U501: moved to B.Cu
- moved U302 347.3 mm to (323.3, 52.4), turned to -90 degrees
- moved R304 330.6 mm to (315.3, 49.8), turned to -90 degrees
- moved R319 327.2 mm to (317.3, 49.8), turned to -90 degrees
- moved R303 325.8 mm to (311.2, 49.8), turned to -90 degrees
- moved R306 322.6 mm to (307.2, 57.1), turned to -90 degrees
- moved R318 322.4 mm to (313.3, 49.8), turned to -90 degrees
- moved R302 321.0 mm to (307.2, 49.8), turned to -90 degrees
- moved R305 317.9 mm to (303.1, 57.1), turned to -90 degrees
- moved R317 317.7 mm to (309.2, 49.8), turned to -90 degrees
- moved R301 316.3 mm to (303.1, 49.8), turned to -90 degrees
- moved R320 314.6 mm to (305.1, 57.1), turned to -90 degrees
- moved R307 314.0 mm to (311.2, 57.1), turned to -90 degrees
- moved R316 312.9 mm to (305.1, 49.8), turned to -90 degrees
- moved R322 310.5 mm to (313.2, 57.1), turned to -90 degrees
- moved R321 305.8 mm to (309.2, 57.1), turned to -90 degrees
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Routing:
- net /Thermistors/TH_3_D: track 0.00 -> 101.3 mm, vias 0 -> 4
- net /Thermistors/TH_3_C: track 0.00 -> 98.8 mm, vias 0 -> 4
- net /Thermistors/TH_3_A: track 0.00 -> 97.4 mm, vias 0 -> 4
- net /Thermistors/TH_3_B: track 0.00 -> 93.5 mm, vias 0 -> 4
- net /ADBMS1818/C1: track 0.00 -> 83.9 mm, vias 0 -> 1
- net /ADBMS1818/C13: track 0.00 -> 74.0 mm, vias 0 -> 1
- net /ADBMS1818/C2: track 0.00 -> 69.1 mm, vias 0 -> 1
- net GND: track 0.00 -> 66.4 mm, vias 0 -> 41
- net /ADBMS1818/C3: track 0.00 -> 63.5 mm, vias 0 -> 1
- net /ADBMS1818/C12: track 0.00 -> 59.7 mm, vias 0 -> 1
- net /ADBMS1818/C11: track 0.00 -> 52.5 mm, vias 0 -> 1
- net /ADBMS1818/C4: track 0.00 -> 51.5 mm, vias 0 -> 1
- net /Thermistors/TH_1_A: track 0.00 -> 51.2 mm, vias 0 -> 2
- net /Thermistors/TH_5_A: track 0.00 -> 50.9 mm, vias 0 -> 2
- net /ADBMS1818/C14: track 0.00 -> 47.2 mm, vias 0 -> 1
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- added copper zone on In2.Cu, net +5V
- added copper zone on F.Cu, net Net-(U601-IND)
- added copper zone on F.Cu, net Net-(U601-SW)
- added copper zone on F.Cu, net Net-(U602-IND)
- added copper zone on F.Cu, net Net-(U602-SW)
Other:
- outline, holes or cut-outs redrawn
- board text added: "${REFERENCE}"
- board text added: "C1001"
- board text added: "C701"
- board text added: "D1001"
- board text added: "F1001"
- board text added: "F1201"
- board text added: "F701"
- board text added: "R1202"
- board text added: "R1203"
- board text added: "R702"
- board text added: "R703"
- board text added: "U301"

Commit message: add stm layout
Parts:
- added R301: 100k, Resistor_SMD:R_0603_1608Metric, F.Cu at (330.8, 124.2)
- added R302: 100k, Resistor_SMD:R_0603_1608Metric, F.Cu at (330.8, 126.7)
- added R303: 100k, Resistor_SMD:R_0603_1608Metric, F.Cu at (330.8, 129.2)
- added R304: 100k, Resistor_SMD:R_0603_1608Metric, F.Cu at (330.8, 131.8)
- added R305: 100k, Resistor_SMD:R_0603_1608Metric, F.Cu at (330.8, 134.3)
- added R306: 100k, Resistor_SMD:R_0603_1608Metric, F.Cu at (334.8, 124.2)
- added R307: 100k, Resistor_SMD:R_0603_1608Metric, F.Cu at (334.8, 126.7)
- added R316: 100k, Resistor_SMD:R_0603_1608Metric, F.Cu at (334.8, 129.2)
- added R317: 100k, Resistor_SMD:R_0603_1608Metric, F.Cu at (334.8, 131.8)
- added R318: 100k, Resistor_SMD:R_0603_1608Metric, F.Cu at (334.8, 134.3)
- added R319: 100k, Resistor_SMD:R_0603_1608Metric, F.Cu at (338.8, 124.2)
- added R320: 100k, Resistor_SMD:R_0603_1608Metric, F.Cu at (338.8, 126.7)
- added R321: 100k, Resistor_SMD:R_0603_1608Metric, F.Cu at (338.8, 129.2)
- added R322: 100k, Resistor_SMD:R_0603_1608Metric, F.Cu at (338.8, 131.8)
- added TP905: TestPoint, TestPoint:TestPoint_Pad_1.0x1.0mm, F.Cu at (330.3, 139.0)
- added TP906: TestPoint, TestPoint:TestPoint_Pad_1.0x1.0mm, F.Cu at (330.3, 142.1)
- added TP907: TestPoint, TestPoint:TestPoint_Pad_1.0x1.0mm, F.Cu at (330.3, 145.1)
- added TP912: TestPoint, TestPoint:TestPoint_Pad_1.0x1.0mm, F.Cu at (330.3, 148.2)
- added TP913: TestPoint, TestPoint:TestPoint_Pad_1.0x1.0mm, F.Cu at (330.3, 151.2)
- added TP914: TestPoint, TestPoint:TestPoint_Pad_1.0x1.0mm, F.Cu at (333.4, 139.0)
- added TP919: TestPoint, TestPoint:TestPoint_Pad_1.0x1.0mm, F.Cu at (333.4, 142.1)
- added TP920: TestPoint, TestPoint:TestPoint_Pad_1.0x1.0mm, F.Cu at (333.4, 145.1)
- added TP921: TestPoint, TestPoint:TestPoint_Pad_1.0x1.0mm, F.Cu at (333.4, 148.2)
- added TP926: TestPoint, TestPoint:TestPoint_Pad_1.0x1.0mm, F.Cu at (333.4, 151.2)
- added TP927: TestPoint, TestPoint:TestPoint_Pad_1.0x1.0mm, F.Cu at (336.4, 139.0)
- added TP928: TestPoint, TestPoint:TestPoint_Pad_1.0x1.0mm, F.Cu at (336.4, 142.1)
- added TP929: TestPoint, TestPoint:TestPoint_Pad_1.0x1.0mm, F.Cu at (336.4, 145.1)
- added TP930: TestPoint, TestPoint:TestPoint_Pad_1.0x1.0mm, F.Cu at (336.4, 148.2)
- added U302: MAX14661ETI+T, BAD_LIB:21-0139I_T2844-1_MXM, F.Cu at (344.0, 126.1)
- added kibuzzard-690D526F: G***, kibuzzard-690D526F, F.Cu at (308.0, 69.6)
- moved C405 233.8 mm to (328.3, 83.1), turned to -90 degrees
- moved C404 232.4 mm to (326.7, 83.1), turned to -90 degrees
- moved R401 228.5 mm to (327.4, 79.3), turned to 180 degrees
- moved R402 225.7 mm to (327.5, 80.8)
- moved C403 222.5 mm to (316.8, 80.2), turned to 90 degrees
- moved R408 222.4 mm to (325.5, 67.1), turned to 90 degrees
- moved J402 219.7 mm to (317.9, 63.9), turned to 90 degrees
- moved R405 219.7 mm to (322.8, 61.6), turned to 180 degrees
- moved R407 219.7 mm to (322.8, 63.2)
- moved Q401 216.5 mm to (323.5, 70.0)
- moved R406 210.0 mm to (313.1, 65.3)
- moved C407 207.7 mm to (302.7, 66.4), turned to -90 degrees
- moved D401 205.1 mm to (323.0, 66.6), turned to 180 degrees
- moved SW401 201.0 mm to (298.4, 67.4), turned to -90 degrees
- moved U402 200.7 mm to (321.8, 80.1)
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Connections:
- J401 pad 2: /STM32/SWDIO -> /STM32/SWCLK
- J401 pad 3: /STM32/SWCLK -> /STM32/SWDIO
Routing:
- net /MUX_SDA: track 0.00 -> 45.0 mm
- net /MUX_SCL: track 0.00 -> 40.8 mm
- net GND: track 66.4 -> 101.0 mm, vias 41 -> 64
- net +3.3V: track 18.0 -> 42.0 mm, vias 44 -> 53
- net Net-(J402-D--PadA7): track 0.00 -> 16.4 mm, vias 0 -> 2
- net Net-(C412-Pad2): track 0.00 -> 15.6 mm
- net Net-(J402-D+-PadA6): track 0.00 -> 14.5 mm, vias 0 -> 4
- net Net-(D401-A): track 0.00 -> 13.5 mm
- net /STM32/RXCAN: track 0.00 -> 12.4 mm
- net /STM32/SWDIO: track 0.00 -> 12.1 mm
- net /STM32/SWCLK: track 0.00 -> 11.3 mm
- net /STM32/TXCAN: track 0.00 -> 11.0 mm
- net /STM32/RESET: track 0.00 -> 9.78 mm, vias 0 -> 2
- net /STM32/D+: track 0.00 -> 6.40 mm
- net Net-(U401-PF0): track 0.00 -> 5.77 mm
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Other:
- copper layers 4 -> 6
