File: Hardware/BMS/cell_tps.kicad_sch (KiCad schematic)
At the start: 15 parts

Commit message: BMS updates, power/fet final updates
Parts:
- TP801, TP802, TP803, TP804, TP805, TP806, TP807, TP808, TP809, TP810, TP811, TP812, TP813, TP814, TP815: footprint TestPoint:TestPoint_Pad_1.0x1.0mm -> TestPoint:TestPoint_Keystone_5019_Miniature

Commit message: bms gotten to 0 unrouted traces!
Parts:
- removed TP801: TestPoint, TestPoint:TestPoint_Keystone_5019_Miniature, symbol Connector:TestPoint
Other:
- moved on the sheet: TP802, TP803, TP804, TP805, TP806, TP807, TP808, TP809, TP810, TP811, TP812, TP813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
