File: Hardware/BMS/leds.kicad_sch (KiCad schematic)
At the start: 24 parts

Commit message: bms gotten to 0 unrouted traces!
Parts:
- removed D1107: LED_0805_Amber, footprints:LED_0805_OEM, symbol formula:LED_0805_Amber
- added D1107: WHITE, LED_SMD:LED_0805_2012Metric, symbol Device:LED
Connections:
- net BMS_HEARTBEAT: now also D1107.2 (A)
- net OT: now also D1101.2 (A); no longer D1106.2 (A)
- net OV: now also D1106.2 (A); no longer D1101.2 (A)
- net UT: now also D1104.2 (A); no longer D1109.2 (A)
- net UV: now also D1109.2 (A); no longer D1104.2 (A)
- net at R1107.1: now also D1107.1 (K)
Changed lines of the file:
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@@
-		)
-	)
-	(hierarchical_label "OT"
-		(shape input)
-		(at 81.28 33.02 180)
-		(effects
-			(font
-				(size 1.27 1.27)
-			)
-			(justify right)
 		)
 	)
@@
 		)
 	)
+	(hierarchical_label "UT"
+		(shape input)
+		(at 58.42 33.02 180)
+		(effects
+			(font
+				(size 1.27 1.27)
+			)
+			(justify right)
+		)
+	)
 	(hierarchical_label "USB_C_COMS"
 		(shape input)
@@
 		)
 	)
+	(hierarchical_label "UV"
+		(shape input)
+		(at 106.68 33.02 180)
+		(effects
+			(font
+				(size 1.27 1.27)
+			)
+			(justify right)
+		)
+	)
 	(hierarchical_label "MUX1_COMS"
 		(shape input)
@@
 	(hierarchical_label "OV"
 		(shape input)
-		(at 33.02 33.02 180)
-		(effects
-			(font
-				(size 1.27 1.27)
-			)
-			(justify right)
-		)
-	)
-	(hierarchical_label "UV"
-		(shape input)
-		(at 58.42 33.02 180)
+		(at 81.28 33.02 180)
 		(effects
 			(font
@@
 		)
 	)
+	(hierarchical_label "OT"
+		(shape input)
+		(at 33.02 33.02 180)
+		(effects
+			(font
+				(size 1.27 1.27)
+			)
+			(justify right)
+		)
+	)
 	(hierarchical_label "ERROR"
 		(shape input)
 		(at 134.62 33.02 180)
-		(effects
-			(font
-				(size 1.27 1.27)
-			)
-			(justify right)
-		)
-	)
-	(hierarchical_label "UT"
-		(shape input)
-		(at 106.68 33.02 180)
 		(effects
 			(font
@@
 	)
 	(symbol
+		(lib_id "Device:LED")
+		(at 85.09 101.6 90)
+		(unit 1)
+		(exclude_from_sim no)
+		(in_bom yes)
+		(on_board yes)
+		(dnp no)
+		(property "Reference" "D1107"
+			(at 86.614 100.33 90)
+			(effects
+				(font
+					(size 1.27 1.27)
+				)
+				(justify right)
+			)
+		)
+		(property "Value" "WHITE"
+			(at 86.868 102.108 90)
+			(effects
+				(font
+					(size 1.27 1.27)
+				)
+				(justify right)
+			)
+		)
+		(property "Footprint" "LED_SMD:LED_0805_2012Metric"
+			(at 85.09 101.6 0)
+			(effects
+				(font
+					(size 1.27 1.27)
+				)
+				(hide yes)
+			)
+		)
+		(property "Datasheet" "~"
+			(at 85.09 101.6 0)
+			(effects
+				(font
+					(size 1.27 1.27)
+				)
+				(hide yes)
+			)
+		)
+		(property "Description" "Light emitting diode"
+			(at 85.09 101.6 0)
+			(effects
+				(font
+					(size 1.27 1.27)
+				)
+				(hide yes)
+			)
+		)
+		(pin "2"
+		)
+		(pin "1"
+		)
+		(instances
+			(project "bms"
+				(path "/36848c1b-92a5-46b0-877b-0db2387c679c/f65c4f1e-6852-4d59-9c03-643ed066f793/e0ab8427-e77b-4bff-9ce4-fd9b0c7b1819"
+					(reference "D1107")
+					(unit 1)
+				)
+			)
+		)
+	)
+	(symbol
 		(lib_id "formula:LED_0805_Red")
 		(at 137.16 36.83 90)
@@
 					(unit 1)
 				)
-			)
-		)
-	)
-	(symbol
-		(lib_id "formula:LED_0805_Amber")
-		(at 85.09 101.6 90)
-		(unit 1)
-		(exclude_from_sim no)
-		(in_bom yes)
-		(on_board yes)
-		(dnp no)
-		(fields_autoplaced yes)
-		(property "Reference" "D1107"
-			(at 88.9 101.9301 90)
-			(effects
-				(font
-					(size 1.27 1.27)
-				)
-				(justify right)
-			)
-		)
-		(property "Value" "LED_0805_Amber"
-			(at 88.9 104.4701 90)
-			(effects
-				(font
-					(size 1.27 1.27)
-				)
-				(justify right)
-			)
-		)
-		(property "Footprint" "footprints:LED_0805_OEM"
-			(at 85.09 104.14 0)
-			(effects
-				(font
-					(size 1.27 1.27)
-				)
-				(hide yes)
-			)
-		)
-		(property "Datasheet" "https://media.digikey.com/pdf/Data%20Sheets/Chicago%20Miniature%20Lamps%20PDFs/CMDA5_Series_Rev_Aug_2014.pdf"
-			(at 82.55 101.6 0)
-			(effects
-				(font
-					(size 1.27 1.27)
-				)
-				(hide yes)
-			)
-		)
-		(property "Description" "LED, Amber, 1.9V, 20mA, 0805"
-			(at 85.09 101.6 0)
-			(effects
-				(font
-					(size 1.27 1.27)
-				)
-				(hide yes)
-			)
-		)
-		(property "MFN" "DK"
-			(at 85.09 101.6 0)
-			(effects
-				(font
-					(size 1.524 1.524)
-				)
-				(hide yes)
-			)
-		)
-		(property "MPN" "L71517CT-ND"
-			(at 85.09 101.6 0)
-			(effects
-				(font
-					(size 1.524 1.524)
-				)
-				(hide yes)
-			)
-		)
-		(property "PurchasingLink" "https://www.digikey.com/product-detail/en/visual-communications-company-vcc/CMDA5DY7D1S/L71517CT-ND/614867"
-			(at 72.39 91.44 0)
-			(effects
-				(font
-					(size 1.524 1.524)
-				)
-				(hide yes)
-			)
-		)
-		(pin "2"
-		)
-		(pin "1"
-		)
-		(instances
-			(project "bms"
-				(path "/36848c1b-92a5-46b0-877b-0db2387c679c/f65c4f1e-6852-4d59-9c03-643ed066f793/e0ab8427-e77b-4bff-9ce4-fd9b0c7b1819"
-					(reference "D1107")
-					(unit 1)
-				)
