File: Hardware/BMS/thermistors.kicad_sch (KiCad schematic)
At the start: 45 parts, among them J301 Conn_02x09_Counter_Clockwise, J302 Conn_02x09_Counter_Clockwise, U301 MAX14661ETI+T, U302 MAX14661ETI+T

Commit message: bms gotten to 0 unrouted traces!
Connections:
- net TH_7_A: now also U302.21 (AB09); no longer U302.18 (AB12)
- net TH_7_B: now also U302.20 (AB10); no longer U302.19 (AB11)
- net TH_7_C: now also U302.19 (AB11); no longer U302.20 (AB10)
- net TH_7_D: now also U302.18 (AB12); no longer U302.21 (AB09)
Other:
- sheet Thermistor Test Points ports: added TH_8_A, TH_8_B; removed none
Changed lines of the file:
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@@
 	(wire
 		(pts
-			(xy 143.51 138.43) (xy 143.51 135.89)
-		)
-		(stroke
-			(width 0)
-			(type default)
-		)
-	)
-	(wire
-		(pts
 			(xy 66.04 119.38) (xy 66.04 132.08)
 		)
@@
 	(wire
 		(pts
-			(xy 143.51 140.97) (xy 143.51 142.24)
+			(xy 143.51 135.89) (xy 143.51 142.24)
 		)
 		(stroke
@@
 	(wire
 		(pts
-			(xy 142.24 140.97) (xy 143.51 140.97)
-		)
-		(stroke
-			(width 0)
-			(type default)
-		)
-	)
-	(wire
-		(pts
 			(xy 199.39 134.62) (xy 201.93 134.62)
 		)
@@
 	(wire
 		(pts
-			(xy 142.24 140.97) (xy 142.24 138.43)
-		)
-		(stroke
-			(width 0)
-			(type default)
-		)
-	)
-	(wire
-		(pts
 			(xy 201.93 64.77) (xy 201.93 67.31)
 		)
@@
 	(wire
 		(pts
-			(xy 142.24 138.43) (xy 143.51 138.43)
-		)
-		(stroke
-			(width 0)
-			(type default)
-		)
-	)
-	(wire
-		(pts
 			(xy 55.88 73.66) (xy 66.04 73.66)
 		)
@@
 		)
 	)
+	(label "TH_7_D"
+		(at 154.94 130.81 180)
+		(effects
+			(font
+				(size 1.27 1.27)
+			)
+			(justify right bottom)
+		)
+	)
 	(label "TH_2_C"
 		(at 91.44 59.69 180)
@@
 		)
 	)
+	(label "TH_7_B"
+		(at 154.94 125.73 180)
+		(effects
+			(font
+				(size 1.27 1.27)
+			)
+			(justify right bottom)
+		)
+	)
 	(label "TH_2_D"
 		(at 241.3 88.9 180)
@@
 	)
 	(label "THERM_AMBIENT"
-		(at 142.24 138.43 180)
+		(at 143.51 138.43 180)
 		(effects
 			(font
@@
 		)
 	)
+	(label "TH_7_A"
+		(at 154.94 123.19 180)
+		(effects
+			(font
+				(size 1.27 1.27)
+			)
+			(justify right bottom)
+		)
+	)
 	(label "TH_7_D"
 		(at 266.7 101.6 0)
@@
 		)
 	)
-	(label "TH_7_A"
-		(at 154.94 130.81 180)
-		(effects
-			(font
-				(size 1.27 1.27)
-			)
-			(justify right bottom)
-		)
-	)
 	(label "TH_3_B"
 		(at 91.44 72.39 180)
@@
 		)
 	)
-	(label "TH_7_C"
-		(at 154.94 125.73 180)
-		(effects
-			(font
-				(size 1.27 1.27)
-			)
-			(justify right bottom)
-		)
-	)
 	(label "TH_2_D"
 		(at 43.18 73.66 180)
@@
 		)
 	)
+	(label "TH_7_C"
+		(at 154.94 128.27 180)
+		(effects
+			(font
+				(size 1.27 1.27)
+			)
+			(justify right bottom)
+		)
+	)
 	(label "TH_4_B"
 		(at 91.44 77.47 180)
@@
 		)
 	)
+	(label "THERM_AMBIENT"
+		(at 266.7 107.95 0)
+		(effects
+			(font
+				(size 1.27 1.27)
+			)
+			(justify left bottom)
+		)
+	)
 	(label "TH_7_A"
 		(at 90.17 151.13 180)
@@
 		)
 	)
-	(label "TH_7_D"
-		(at 154.94 123.19 180)
-		(effects
-			(font
-				(size 1.27 1.27)
-			)
-			(justify right bottom)
-		)
-	)
 	(label "TH_5_D"
 		(at 43.18 119.38 180)
@@
 		)
 	)
-	(label "TH_7_B"
-		(at 154.94 128.27 180)
-		(effects
-			(font
-				(size 1.27 1.27)
-			)
-			(justify right bottom)
-		)
-	)
 	(label "TH_6_D"
 		(at 154.94 120.65 180)
@@
 		)
 	)
+	(hierarchical_label "THERM_BUSBAR"
+		(shape input)
+		(at 266.7 105.41 0)
+		(effects
+			(font
+				(size 1.27 1.27)
+			)
+			(justify left)
+		)
+	)
 	(hierarchical_label "SCL"
 		(shape output)
@@
 			(effects
 				(font
+					(size 1.27 1.27)
+				)
+				(justify right)
+			)
+		)
+		(pin "TH_8_A" input
+			(at 266.7 105.41 0)
+			(effects
+				(font
+					(size 1.27 1.27)
+				)
+				(justify right)
+			)
+		)
+		(pin "TH_8_B" input
+			(at 266.7 107.95 0)
+			(effects
+				(font
