File: Hardware/BMS/ADBMS1818.kicad_sch (KiCad schematic)
At the start: 6 parts, among them J501 Conn_02x09_Counter_Clockwise, U501 ADBMS1818

Commit message: bms gotten to 0 unrouted traces!
Other:
- sheet Cell Test Points ports: added none; removed CELL0
Changed lines of the file:
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@@
-		)
-	)
-	(label "CELL0"
-		(at 161.29 27.94 180)
-		(effects
-			(font
-				(size 1.27 1.27)
-			)
-			(justify right bottom)
 		)
 	)
@@
 			)
 		)
-		(pin "CELL0" input
-			(at 161.29 27.94 180)
-			(effects
-				(font
-					(size 1.27 1.27)
-				)
-				(justify left)
-			)
-		)

Commit message: fab updates to bms, power board, fet board
Parts:
- added F501: 4A, Fuse:Fuse_1206_3216Metric, symbol Device:Fuse
Connections:
- net BATT+: now also F501.1; no longer J501.18 (Pin_18)
- new net: F501.2, J501.18 (Pin_18)
Changed lines of the file:
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@@
 	(wire
 		(pts
+			(xy 158.75 85.09) (xy 167.64 85.09)
+		)
+		(stroke
+			(width 0)
+			(type default)
+		)
+	)
+	(wire
+		(pts
 			(xy 134.62 40.64) (xy 125.73 40.64)
 		)
@@
 		)
 	)
-	(hierarchical_label "CSB"
+	(hierarchical_label "BATT+"
 		(shape input)
-		(at 265.43 95.25 0)
+		(at 151.13 85.09 180)
 		(effects
 			(font
 				(size 1.27 1.27)
 			)
-			(justify left)
+			(justify right)
 		)
 	)
-	(hierarchical_label "BATT+"
+	(hierarchical_label "CSB"
 		(shape input)
-		(at 167.64 85.09 180)
+		(at 265.43 95.25 0)
 		(effects
 			(font
 				(size 1.27 1.27)
 			)
-			(justify right)
+			(justify left)
 		)
 	)
@@
 					(unit 1)
 				)
+			)
+		)
+	)
+	(symbol
+		(lib_id "Device:Fuse")
+		(at 154.94 85.09 90)
+		(unit 1)
+		(exclude_from_sim no)
+		(in_bom yes)
+		(on_board yes)
+		(dnp no)
+		(property "Reference" "F501"
+			(at 154.94 87.122 90)
+			(effects
+				(font
+					(size 1.27 1.27)
+				)
+			)
+		)
+		(property "Value" "4A"
+			(at 154.94 83.058 90)
+			(effects
+				(font
+					(size 1.27 1.27)
+				)
+			)
+		)
+		(property "Footprint" "Fuse:Fuse_1206_3216Metric"
+			(at 154.94 86.868 90)
+			(effects
+				(font
+					(size 1.27 1.27)
+				)
+				(hide yes)
+			)
+		)
+		(property "Datasheet" "~"
+			(at 154.94 85.09 0)
+			(effects
+				(font
+					(size 1.27 1.27)
+				)
+				(hide yes)
+			)
+		)
+		(property "Description" "Fuse, 4A, 72V, Fast Blow"
+			(at 154.94 85.09 0)
+			(effects
+				(font
+					(size 1.27 1.27)
+				)
+				(hide yes)
+			)
+		)
+		(pin "2"
+		)
+		(pin "1"
+		)
+		(instances
+			(project ""
+				(path "/36848c1b-92a5-46b0-877b-0db2387c679c/826e6c70-848d-4f04-803e-a5eb891d5409"
+					(reference "F501")
+					(unit 1)
+				)
