File: Hardware/BMS/bms.kicad_sch (KiCad schematic)
At the start: 31 parts, among them J101 Conn_02x02_Counter_Clockwise, J102 Conn_01x02, J103 Conn_02x05_Top_Bottom, U101 TSC2011IST, U102 74AHC1G08, U103 LTV-356T

Commit message: BMS updates, power/fet final updates
Parts:
- J102: footprint Connector_Molex:Molex_Nano-Fit_105313-xx02_1x02_P2.50mm_Horizontal -> Connector_Molex:Molex_Micro-Fit_3.0_43650-0200_1x02_P3.00mm_Horizontal
Changed lines of the file:
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@@
 			)
 		)
-		(property "Footprint" "Connector_Molex:Molex_Nano-Fit_105313-xx02_1x02_P2.50mm_Horizontal"
+		(property "Footprint" "Connector_Molex:Molex_Micro-Fit_3.0_43650-0200_1x02_P3.00mm_Horizontal"
 			(at 123.19 137.16 0)
 			(effects

Commit message: bms gotten to 0 unrouted traces!
Parts:
- added R109: 24k, Resistor_SMD:R_0603_1608Metric, symbol Device:R
- added R110: 750, Resistor_SMD:R_0603_1608Metric, symbol Device:R
Connections:
- net +3.3V: now also R109.2
- net GND: now also R110.1; no longer U101.3 (VREF2), U101.7 (VREF1)
- new net: R109.1, R110.2, U101.3 (VREF2), U101.7 (VREF1)
- no-connect marks 1 -> 0
Other:
- added sheet Fans (fans.kicad_sch)
- sheet Power ports: added PS_EN; removed none
- sheet STM32 ports: added FAN_EXT, FAN_INT; removed none
- note added: "TODO: FAN STUFF"
- note removed: "TODO: Testpoints LEDs"

Commit message: fab updates to bms, power board, fet board
Parts:
- D103: value BLUE -> WHITE
Other:
- sheet ADBMS1818 ports: added +3.3V; removed none
Changed lines of the file:
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@@
 	(wire
 		(pts
-			(xy 226.06 67.31) (xy 226.06 59.69)
+			(xy 226.06 64.77) (xy 226.06 59.69)
 		)
 		(stroke
@@
 	(wire
 		(pts
-			(xy 232.41 62.23) (xy 232.41 59.69)
+			(xy 232.41 60.96) (xy 232.41 59.69)
 		)
 		(stroke
@@
 	(wire
 		(pts
+			(xy 219.71 68.58) (xy 237.49 68.58)
+		)
+		(stroke
+			(width 0)
+			(type default)
+		)
+	)
+	(wire
+		(pts
 			(xy 123.19 158.75) (xy 123.19 160.02)
 		)
@@
 	(wire
 		(pts
+			(xy 219.71 59.69) (xy 219.71 68.58)
+		)
+		(stroke
+			(width 0)
+			(type default)
+		)
+	)
+	(wire
+		(pts
 			(xy 67.31 176.53) (xy 78.74 176.53)
 		)
@@
 	(wire
 		(pts
-			(xy 237.49 62.23) (xy 232.41 62.23)
+			(xy 237.49 60.96) (xy 232.41 60.96)
 		)
 		(stroke
@@
 	(wire
 		(pts
-			(xy 237.49 67.31) (xy 226.06 67.31)
+			(xy 237.49 64.77) (xy 226.06 64.77)
 		)
 		(stroke
@@
 			)
 		)
-		(property "Value" "BLUE"
+		(property "Value" "WHITE"
 			(at 151.638 177.038 90)
 			(effects
@@
 	)
 	(symbol
+		(lib_id "power:+3.3V")
+		(at 219.71 59.69 0)
+		(unit 1)
+		(exclude_from_sim no)
+		(in_bom yes)
+		(on_board yes)
+		(dnp no)
+		(fields_autoplaced yes)
+		(property "Reference" "#PWR0134"
+			(at 219.71 63.5 0)
+			(effects
+				(font
+					(size 1.27 1.27)
+				)
+				(hide yes)
+			)
+		)
+		(property "Value" "+3.3V"
+			(at 219.71 54.61 0)
+			(effects
+				(font
+					(size 1.27 1.27)
+				)
+			)
+		)
+		(property "Footprint" ""
+			(at 219.71 59.69 0)
+			(effects
+				(font
+					(size 1.27 1.27)
+				)
+				(hide yes)
+			)
+		)
+		(property "Datasheet" ""
+			(at 219.71 59.69 0)
+			(effects
+				(font
+					(size 1.27 1.27)
+				)
+				(hide yes)
+			)
+		)
+		(property "Description" "Power symbol creates a global label with name \"+3.3V\""
+			(at 219.71 59.69 0)
+			(effects
+				(font
+					(size 1.27 1.27)
+				)
+				(hide yes)
+			)
+		)
+		(pin "1"
+		)
+		(instances
+			(project "bms"
+				(path "/36848c1b-92a5-46b0-877b-0db2387c679c"
+					(reference "#PWR0134")
+					(unit 1)
+				)
+			)
+		)
+	)
+	(symbol
 		(lib_id "Device:R")
 		(at 29.21 176.53 180)
@@
 		)
 		(pin "+5V" input
-			(at 237.49 67.31 180)
+			(at 237.49 64.77 180)
 			(effects
 				(font
@@
 		)
 		(pin "BATT+" input
-			(at 237.49 62.23 180)
+			(at 237.49 60.96 180)
 			(effects
 				(font
@@
 			)
 		)
+		(pin "+3.3V" input
+			(at 237.49 68.58 180)
+			(effects
+				(font
+					(size 1.27 1.27)
+				)
+				(justify left)
+			)
+		)

Commit message: created sponsorship coaster
Other:
- note removed: "TODO: FAN STUFF"
Changed lines of the file:
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@@
-		)
-	)
-	(text "TODO:\nFAN STUFF"
-		(exclude_from_sim no)
-		(at 82.296 91.694 0)
-		(effects
-			(font
-				(size 5 5)
-			)
 		)
 	)
