File: Hardware/BMS/power.kicad_sch (KiCad schematic)
At the start: 33 parts, among them Q601 SQ2337ES

Commit message: bms gotten to 0 unrouted traces!
Parts:
- added C619: 2.2uF, Capacitor_SMD:C_0603_1608Metric, symbol Device:C
- added R610: 100k, Resistor_SMD:R_0603_1608Metric, symbol Device:R
Connections:
- net +BATT: now also Q601.2 (S); no longer Q601.3 (D)
- net GND: now also C619.2
- net PS_EN: now also Q601.3 (D); no longer Q601.2 (S)
- net at D601.2 (A), R603.2, R604.1: now also R610.2; no longer Q601.1 (G)
- new net: C619.1, Q601.1 (G), R610.1
Other:
- moved on the sheet: D601, Q601, R603, R604

Commit message: fab updates to bms, power board, fet board
Parts:
- C601, C610, C619: footprint Capacitor_SMD:C_0603_1608Metric -> Capacitor_SMD:C_0805_2012Metric
Changed lines of the file:
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@@
 			)
 		)
-		(property "Footprint" "Capacitor_SMD:C_0603_1608Metric"
+		(property "Footprint" "Capacitor_SMD:C_0805_2012Metric"
 			(at 37.7952 64.77 0)
 			(effects
@@
 			)
 		)
-		(property "Footprint" "Capacitor_SMD:C_0603_1608Metric"
+		(property "Footprint" "Capacitor_SMD:C_0805_2012Metric"
 			(at 55.5752 143.51 0)
 			(effects
@@
 			)
 		)
-		(property "Footprint" "Capacitor_SMD:C_0603_1608Metric"
+		(property "Footprint" "Capacitor_SMD:C_0805_2012Metric"
 			(at 163.5252 64.77 0)
 			(effects

Commit message: CAN library working with dbc, yml, for extended and standard IDs. Core finalized. BMS firmware bringup started
Parts:
- C602, C605, C611, C614: value 100pf -> 0.1uF
Other:
- note added: "WRONG!!"
Changed lines of the file:
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@@
 		)
 	)
+	(text "WRONG!!"
+		(exclude_from_sim no)
+		(at 108.966 57.404 0)
+		(effects
+			(font
+				(size 3 3)
+				(thickness 0.6)
+				(bold yes)
+			)
+		)
+	)
 	(text "3.3V Buck Converter"
 		(exclude_from_sim no)
@@
 		)
 	)
+	(text "WRONG!!"
+		(exclude_from_sim no)
+		(at 164.338 71.628 0)
+		(effects
+			(font
+				(size 3 3)
+				(thickness 0.6)
+				(bold yes)
+			)
+		)
+	)
 	(text "ADBMS Datasheet pg71"
 		(exclude_from_sim no)
@@
 		)
 	)
+	(text "WRONG!!"
+		(exclude_from_sim no)
+		(at 224.028 57.912 0)
+		(effects
+			(font
+				(size 3 3)
+				(thickness 0.6)
+				(bold yes)
+			)
+		)
+	)
+	(text "WRONG!!"
+		(exclude_from_sim no)
+		(at 36.322 65.278 0)
+		(effects
+			(font
+				(size 3 3)
+				(thickness 0.6)
+				(bold yes)
+			)
+		)
+	)
 	(text "POWER"
 		(exclude_from_sim no)
@@
 			)
 		)
-		(property "Value" "100pf"
+		(property "Value" "0.1uF"
 			(at 96.52 60.452 0)
 			(effects
@@
 			)
 		)
-		(property "Value" "100pf"
+		(property "Value" "0.1uF"
 			(at 222.25 60.452 0)
 			(effects
@@
 			)
 		)
-		(property "Value" "100pf"
+		(property "Value" "0.1uF"
 			(at 40.64 74.422 0)
 			(effects
@@
 			)
 		)
-		(property "Value" "100pf"
+		(property "Value" "0.1uF"
 			(at 166.37 74.422 0)
 			(effects

Commit message: created sponsorship coaster
Other:
- note removed: "WRONG!!"
Changed lines of the file:
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@@
-		)
-	)
-	(text "WRONG!!"
-		(exclude_from_sim no)
-		(at 108.966 57.404 0)
-		(effects
-			(font
-				(size 3 3)
-				(thickness 0.6)
-				(bold yes)
-			)
 		)
 	)
@@
 			(font
 				(size 3 3)
-			)
-		)
-	)
-	(text "WRONG!!"
-		(exclude_from_sim no)
-		(at 164.338 71.628 0)
-		(effects
-			(font
-				(size 3 3)
-				(thickness 0.6)
-				(bold yes)
 			)
 		)
@@
 			)
 		)
-	)
-	(text "WRONG!!"
-		(exclude_from_sim no)
-		(at 224.028 57.912 0)
-		(effects
-			(font
-				(size 3 3)
-				(thickness 0.6)
-				(bold yes)
-			)
-		)
-	)
-	(text "WRONG!!"
-		(exclude_from_sim no)
-		(at 36.322 65.278 0)
-		(effects
-			(font
-				(size 3 3)
-				(thickness 0.6)
-				(bold yes)
-			)
-		)
