File: Hardware/Power Board/Power Board.kicad_sch (KiCad schematic)
At the start: 31 parts, among them J1 Conn_02x09_Counter_Clockwise, J10 Conn_01x05_MountingPin, J2 Conn_02x09_Counter_Clockwise, J3 Conn_02x09_Counter_Clockwise, J4 Conn_01x05_MountingPin, J5 Conn_01x05_MountingPin, J6 Conn_01x05_MountingPin, J7 Conn_01x05_MountingPin, J8 Conn_01x05_MountingPin, J9 Conn_01x05_MountingPin

Commit message: BMS updates, power/fet final updates
Parts:
- J1, J2, J3: footprint Connector_PinSocket_2.54mm:PinSocket_2x09_P2.54mm_Vertical -> Connector_PinHeader_2.54mm:PinHeader_2x09_P2.54mm_Vertical
