File: Hardware/Core/flight-core/cube_1.kicad_sch (KiCad schematic)
At the start: 17 parts, among them J10 Conn_01x06, J11 Conn_01x04_Socket, J12 Conn_01x04_Socket, J13 Conn_01x06, J14 MicroFit_VT_3, J8 MicroFit_VT_3, J9 Cube Orange Plus Female Header, Q1 MMBF170, Q2 MMBF170, Q3 MMBF170

Commit message: adding passive buzzer, moving buzzer to gpio pin
Parts:
- added LS1: CST-951AP, obad_footprints:CUI_CST-951AP, symbol OlinBAD:CST-951AP
Connections:
- net ALARM: no longer Q3.1 (G)
- net GND: now also LS1.M
- net BUZZER: now reaches J9.54
- net BUZZER: now also Q3.1 (G)
- net at Q3.2 (S): now also LS1.P
- no-connect marks 51 -> 50
Changed lines of the file:
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@@
 	(text "BUZZER"
 		(exclude_from_sim no)
-		(at 265.43 148.59 0)
+		(at 279.4 106.68 0)
 		(effects
 			(font
@@
 	)
 	(no_connect
-		(at 96.52 116.84)
-	)
-	(no_connect
 		(at 96.52 55.88)
 	)
@@
 	(wire
 		(pts
+			(xy 274.32 133.35) (xy 274.32 135.89)
+		)
+		(stroke
+			(width 0)
+			(type default)
+		)
+	)
+	(wire
+		(pts
 			(xy 45.72 152.4) (xy 52.07 152.4)
 		)
@@
 		)
 	)
+	(wire
+		(pts
+			(xy 274.32 146.05) (xy 274.32 148.59)
+		)
+		(stroke
+			(width 0)
+			(type default)
+		)
+	)
 	(bus
 		(pts
@@
 		)
 	)
-	(label "UART_TELEM2_RX"
-		(at 227.33 73.66 180)
+	(label "BUZZER"
+		(at 266.7 128.27 180)
 		(effects
 			(font
@@
 		)
 	)
-	(label "ALARM"
-		(at 266.7 128.27 180)
+	(label "UART_TELEM2_RX"
+		(at 227.33 73.66 180)
 		(effects
 			(font
@@
 		)
 	)
+	(label "BUZZER"
+		(at 96.52 116.84 0)
+		(effects
+			(font
+				(size 1.27 1.27)
+			)
+			(justify left bottom)
+		)
+	)
 	(label "FMU_LED_AMBER"
 		(at 96.52 50.8 0)
@@
 	)
 	(symbol
+		(lib_id "OlinBAD:CST-951AP")
+		(at 274.32 140.97 0)
+		(unit 1)
+		(exclude_from_sim no)
+		(in_bom yes)
+		(on_board yes)
+		(dnp no)
+		(fields_autoplaced yes)
+		(property "Reference" "LS1"
+			(at 278.13 139.947 0)
+			(effects
+				(font
+					(size 1.27 1.27)
+				)
+				(justify left)
+			)
+		)
+		(property "Value" "CST-951AP"
+			(at 278.13 142.487 0)
+			(effects
+				(font
+					(size 1.27 1.27)
+				)
+				(justify left)
+			)
+		)
+		(property "Footprint" "obad_footprints:CUI_CST-951AP"
+			(at 274.32 140.97 0)
+			(effects
+				(font
+					(size 1.27 1.27)
+				)
+				(justify bottom)
+				(hide yes)
+			)
+		)
+		(property "Datasheet" ""
+			(at 274.32 140.97 0)
+			(effects
+				(font
+					(size 1.27 1.27)
+				)
+				(hide yes)
+			)
+		)
+		(property "Description" "Audio Buzzer Magnetic 4Vo-p 6Vo-p 8mA 5Vo-p 85dBA Pin Through Hole Tray"
+			(at 274.32 140.97 0)
+			(effects
+				(font
+					(size 1.27 1.27)
+				)
+				(justify bottom)
+				(hide yes)
+			)
+		)
+		(property "MF" "CUI"
+			(at 274.32 140.97 0)
+			(effects
+				(font
+					(size 1.27 1.27)
+				)
+				(justify bottom)
+				(hide yes)
+			)
+		)
+		(property "PACKAGE" "CUI"
+			(at 274.32 140.97 0)
+			(effects
+				(font
+					(size 1.27 1.27)
+				)
+				(justify bottom)
+				(hide yes)
+			)
+		)
+		(property "PRICE" "0.69 USD"
+			(at 274.32 140.97 0)
+			(effects
+				(font
+					(size 1.27 1.27)
+				)
+				(justify bottom)
+				(hide yes)
+			)
+		)
+		(property "MP" "CST-951AP"
+			(at 274.32 140.97 0)
+			(effects
+				(font
+					(size 1.27 1.27)
+				)
+				(justify bottom)
+				(hide yes)
+			)
+		)
+		(property "AVAILABILITY" "Good"
+			(at 274.32 140.97 0)
+			(effects
+				(font
+					(size 1.27 1.27)
+				)
+				(justify bottom)
+				(hide yes)
+			)
+		)
+		(pin "P"
+		)
+		(pin "M"
+		)
+		(instances
+			(project ""
+				(path "/93f46f4b-cdf5-47ec-af03-96378e73b2e1/5021d7c9-30f6-40e8-9368-2fcfccc5f247"
+					(reference "LS2")
+					(unit 1)
+				)
+				(path "/93f46f4b-cdf5-47ec-af03-96378e73b2e1/b1ca264a-f418-4fe7-a7ba-dc33a197c475"
+					(reference "LS1")
+					(unit 1)
+				)
+			)
+		)
+	)
+	(symbol
 		(lib_id "Connector:Conn_01x04_Socket")
 		(at 171.45 45.72 0)
@@
 					(unit 1)
 				)
+			)
+		)
+	)
+	(symbol
+		(lib_id "power:GND")
+		(at 274.32 148.59 0)
+		(unit 1)
+		(exclude_from_sim no)
+		(in_bom yes)
+		(on_board yes)
+		(dnp no)
+		(fields_autoplaced yes)
+		(property "Reference" "#PWR0447"
+			(at 274.32 154.94 0)
+			(effects
+				(font
+					(size 1.27 1.27)
+				)
+				(hide yes)
+			)
+		)
+		(property "Value" "GND"
+			(at 274.32 153.67 0)
+			(effects
+				(font
+					(size 1.27 1.27)
+				)
+			)
+		)
+		(property "Footprint" ""
+			(at 274.32 148.59 0)
+			(effects
+				(font
+					(size 1.27 1.27)
+				)
+				(hide yes)
+			)
+		)
+		(property "Datasheet" ""
+			(at 274.32 148.59 0)
+			(effects
+				(font
+					(size 1.27 1.27)
+				)
+				(hide yes)
+			)
+		)
+		(property "Description" "Power symbol creates a global label with name \"GND\" , ground"
+			(at 274.32 148.59 0)
+			(effects
+				(font
+					(size 1.27 1.27)
+				)
+				(hide yes)
+			)
+		)
+		(pin "1"
+		)
+		(instances
+			(project ""
+				(path "/93f46f4b-cdf5-47ec-af03-96378e73b2e1/5021d7c9-30f6-40e8-9368-2fcfccc5f247"
+					(reference "#PWR0448")
+					(unit 1)
+				)
+				(path "/93f46f4b-cdf5-47ec-af03-96378e73b2e1/b1ca264a-f418-4fe7-a7ba-dc33a197c475"
+					(reference "#PWR0447")
+					(unit 1)
+				)

Commit message: importeed bms board settings and began rerouting repeater
Parts:
- added TP34, TP36, TP38: TP, footprints:tp_1.6mm, symbol formula:TP
Connections:
- net at J9.56: now also TP38.1 (TP)
- net at J9.58: now also TP36.1 (TP)
- net at J9.60: now also TP34.1 (TP)
- no-connect marks 50 -> 47
