File: Hardware/Core/flight-core/can_repeater.kicad_sch (KiCad schematic)
At the start: 9 parts, among them U6 TCAN1042HGVDRQ1, U7 TCAN1042HGVDRQ1

Commit message: added sense pwr cycle pull down, low side cube mosfets, fixed mosi/miso swap on i/o expander, Rs -> generic, reannotated
Parts:
- renumbered R11 to R12, R12 to R13
