File: Hardware/Core/flight-core/converters.kicad_sch (KiCad schematic)
At the start: 19 parts, among them Q5 DMN10H220L, U57 Fuse_Holder_Blade, U58 5V VCC Current Sensor, U59 18-75V to 5V Converter, U60 Fuse_Holder_Blade, U61 TPS62086RLTR, U62 3.3V VCC Current Sensor

Commit message: added sense pwr cycle pull down, low side cube mosfets, fixed mosi/miso swap on i/o expander, Rs -> generic, reannotated
Parts:
- renumbered C109 to C102, C110 to C103, C111 to C104, C112 to C105, C113 to C106
Changed lines of the file:
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@@
 		(dnp no)
 		(fields_autoplaced yes)
-		(property "Reference" "#PWR0210"
+		(property "Reference" "#PWR0211"
 			(at 49.53 81.28 0)
 			(effects
@@
 			(project "flight-core"
 				(path "/93f46f4b-cdf5-47ec-af03-96378e73b2e1/f120f04e-9926-485a-8729-a726a206f3dc"
-					(reference "#PWR0210")
+					(reference "#PWR0211")
 					(unit 1)
 				)
@@
 		(on_board yes)
 		(dnp no)
-		(property "Reference" "C109"
+		(property "Reference" "C102"
 			(at 61.722 63.754 0)
 			(effects
@@
 			(project ""
 				(path "/93f46f4b-cdf5-47ec-af03-96378e73b2e1/f120f04e-9926-485a-8729-a726a206f3dc"
-					(reference "C109")
+					(reference "C102")
 					(unit 1)
 				)
@@
 		(dnp no)
 		(fields_autoplaced yes)
-		(property "Reference" "#PWR0223"
+		(property "Reference" "#PWR0224"
 			(at 252.73 60.96 0)
 			(effects
@@
 			(project "flight-core"
 				(path "/93f46f4b-cdf5-47ec-af03-96378e73b2e1/f120f04e-9926-485a-8729-a726a206f3dc"
-					(reference "#PWR0223")
+					(reference "#PWR0224")
 					(unit 1)
 				)
@@
 		(dnp no)
 		(fields_autoplaced yes)
-		(property "Reference" "#PWR0219"
+		(property "Reference" "#PWR0220"
 			(at 194.31 102.87 0)
 			(effects
@@
 			(project "flight-core"
 				(path "/93f46f4b-cdf5-47ec-af03-96378e73b2e1/f120f04e-9926-485a-8729-a726a206f3dc"
-					(reference "#PWR0219")
+					(reference "#PWR0220")
 					(unit 1)
 				)
@@
 		(dnp no)
 		(fields_autoplaced yes)
-		(property "Reference" "#PWR0215"
+		(property "Reference" "#PWR0216"
 			(at 139.7 123.19 0)
 			(effects
@@
 			(project "flight-core"
 				(path "/93f46f4b-cdf5-47ec-af03-96378e73b2e1/f120f04e-9926-485a-8729-a726a206f3dc"
-					(reference "#PWR0215")
+					(reference "#PWR0216")
 					(unit 1)
 				)
@@
 		(dnp no)
 		(fields_autoplaced yes)
-		(property "Reference" "#PWR0222"
+		(property "Reference" "#PWR0223"
 			(at 241.3 139.7 0)
 			(effects
@@
 			(project "flight-core"
 				(path "/93f46f4b-cdf5-47ec-af03-96378e73b2e1/f120f04e-9926-485a-8729-a726a206f3dc"
-					(reference "#PWR0222")
+					(reference "#PWR0223")
 					(unit 1)
 				)
@@
 		(dnp no)
 		(fields_autoplaced yes)
-		(property "Reference" "C113"
+		(property "Reference" "C106"
 			(at 245.11 126.9999 0)
 			(effects
@@
 			(project "flight-core"
 				(path "/93f46f4b-cdf5-47ec-af03-96378e73b2e1/f120f04e-9926-485a-8729-a726a206f3dc"
-					(reference "C113")
+					(reference "C106")
 					(unit 1)
 				)
@@
 		(dnp no)
 		(fields_autoplaced yes)
-		(property "Reference" "#PWR0221"
+		(property "Reference" "#PWR0222"
 			(at 241.3 124.46 0)
 			(effects
@@
 			(project "flight-core"
 				(path "/93f46f4b-cdf5-47ec-af03-96378e73b2e1/f120f04e-9926-485a-8729-a726a206f3dc"
-					(reference "#PWR0221")
+					(reference "#PWR0222")
 					(unit 1)
 				)
@@
 		(dnp no)
 		(fields_autoplaced yes)
-		(property "Reference" "#PWR0212"
+		(property "Reference" "#PWR0213"
 			(at 73.66 81.28 0)
 			(effects
@@
 			(project "flight-core"
 				(path "/93f46f4b-cdf5-47ec-af03-96378e73b2e1/f120f04e-9926-485a-8729-a726a206f3dc"
-					(reference "#PWR0212")
+					(reference "#PWR0213")
 					(unit 1)
 				)
@@
 		(dnp no)
 		(fields_autoplaced yes)
-		(property "Reference" "#PWR0211"
+		(property "Reference" "#PWR0212"
 			(at 60.96 81.28 0)
 			(effects
@@
 			(project "flight-core"
 				(path "/93f46f4b-cdf5-47ec-af03-96378e73b2e1/f120f04e-9926-485a-8729-a726a206f3dc"
-					(reference "#PWR0211")
+					(reference "#PWR0212")
 					(unit 1)
 				)
@@
 		(on_board yes)
 		(dnp no)
-		(property "Reference" "#PWR0217"
+		(property "Reference" "#PWR0218"
 			(at 147.32 81.28 0)
 			(effects
@@
 			(project "flight-core"
 				(path "/93f46f4b-cdf5-47ec-af03-96378e73b2e1/f120f04e-9926-485a-8729-a726a206f3dc"
-					(reference "#PWR0217")
+					(reference "#PWR0218")
 					(unit 1)
 				)
@@
 		(dnp no)
 		(fields_autoplaced yes)
-		(property "Reference" "#PWR0218"
+		(property "Reference" "#PWR0219"
 			(at 168.91 58.42 0)
 			(effects
@@
 			(project ""
 				(path "/93f46f4b-cdf5-47ec-af03-96378e73b2e1/f120f04e-9926-485a-8729-a726a206f3dc"
-					(reference "#PWR0218")
+					(reference "#PWR0219")
 					(unit 1)
 				)
@@
 		(dnp no)
 		(fields_autoplaced yes)
-		(property "Reference" "#PWR0216"
+		(property "Reference" "#PWR0217"
 			(at 139.7 138.43 0)
 			(effects
@@
 			(project "flight-core"
 				(path "/93f46f4b-cdf5-47ec-af03-96378e73b2e1/f120f04e-9926-485a-8729-a726a206f3dc"
-					(reference "#PWR0216")
+					(reference "#PWR0217")
 					(unit 1)
 				)
@@
 		(dnp no)
 		(fields_autoplaced yes)
-		(property "Reference" "#PWR0220"
+		(property "Reference" "#PWR0221"
 			(at 223.52 139.7 0)
 			(effects
@@
 			(project "flight-core"
 				(path "/93f46f4b-cdf5-47ec-af03-96378e73b2e1/f120f04e-9926-485a-8729-a726a206f3dc"
-					(reference "#PWR0220")
+					(reference "#PWR0221")
 					(unit 1)
 				)
@@
 		(dnp no)
 		(fields_autoplaced yes)
-		(property "Reference" "C111"
+		(property "Reference" "C104"
 			(at 167.64 76.1999 0)
 			(effects
@@
 			(project "flight-core"
 				(path "/93f46f4b-cdf5-47ec-af03-96378e73b2e1/f120f04e-9926-485a-8729-a726a206f3dc"
-					(reference "C111")
+					(reference "C104")
 					(unit 1)
 				)
@@
 		(on_board yes)
 		(dnp no)
-		(property "Reference" "#PWR0213"
+		(property "Reference" "#PWR0214"
 			(at 93.98 81.28 0)
 			(effects
@@
 			(project "flight-core"
 				(path "/93f46f4b-cdf5-47ec-af03-96378e73b2e1/f120f04e-9926-485a-8729-a726a206f3dc"
-					(reference "#PWR0213")
+					(reference "#PWR0214")
 					(unit 1)
 				)
@@
 		(dnp no)
 		(fields_autoplaced yes)
-		(property "Reference" "C112"
+		(property "Reference" "C105"
 			(at 241.3 82.5499 0)
 			(effects
@@
 			(project "flight-core"
 				(path "/93f46f4b-cdf5-47ec-af03-96378e73b2e1/f120f04e-9926-485a-8729-a726a206f3dc"
-					(reference "C112")
+					(reference "C105")
 					(unit 1)
 				)
@@
 		(dnp no)
 		(fields_autoplaced yes)
-		(property "Reference" "#PWR0214"
+		(property "Reference" "#PWR0215"
 			(at 120.65 138.43 0)
 			(effects
@@
 			(project "flight-core"
 				(path "/93f46f4b-cdf5-47ec-af03-96378e73b2e1/f120f04e-9926-485a-8729-a726a206f3dc"
-					(reference "#PWR0214")
+					(reference "#PWR0215")
 					(unit 1)
 				)
@@
 		(dnp no)
 		(fields_autoplaced yes)
-		(property "Reference" "C110"
+		(property "Reference" "C103"
 			(at 143.51 125.7299 0)
 			(effects
@@
 			(project "flight-core"
 				(path "/93f46f4b-cdf5-47ec-af03-96378e73b2e1/f120f04e-9926-485a-8729-a726a206f3dc"
-					(reference "C110")
-					(unit 1)
-				)
+					(reference "C103")
+					(unit 1)
+				)

Commit message: major component area placement begun, installing place footprints plugin, updating connectors to vertical
Parts:
- renumbered D7 to D22, Q5 to Q20, R50 to R64, R51 to R65, R52 to R66, R53 to R67, R54 to R68, U57 to U56, U58 to U57, U59 to U58, U60 to U59, U61 to U60, U62 to U61
Changed lines of the file:
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@@
 		(dnp no)
 		(fields_autoplaced yes)
-		(property "Reference" "#PWR0211"
+		(property "Reference" "#PWR0241"
 			(at 49.53 81.28 0)
 			(effects
@@
 			(project "flight-core"
 				(path "/93f46f4b-cdf5-47ec-af03-96378e73b2e1/f120f04e-9926-485a-8729-a726a206f3dc"
-					(reference "#PWR0211")
+					(reference "#PWR0241")
 					(unit 1)
 				)
@@
 		(dnp no)
 		(fields_autoplaced yes)
-		(property "Reference" "#PWR0224"
+		(property "Reference" "#PWR0254"
 			(at 252.73 60.96 0)
 			(effects
@@
 			(project "flight-core"
 				(path "/93f46f4b-cdf5-47ec-af03-96378e73b2e1/f120f04e-9926-485a-8729-a726a206f3dc"
-					(reference "#PWR0224")
+					(reference "#PWR0254")
 					(unit 1)
 				)
@@
 		(on_board yes)
 		(dnp no)
-		(property "Reference" "R54"
+		(property "Reference" "R68"
 			(at 223.266 79.502 90)
 			(effects
@@
 			(project "flight-core"
 				(path "/93f46f4b-cdf5-47ec-af03-96378e73b2e1/f120f04e-9926-485a-8729-a726a206f3dc"
-					(reference "R54")
+					(reference "R68")
 					(unit 1)
 				)
@@
 		(dnp no)
 		(fields_autoplaced yes)
-		(property "Reference" "#PWR0220"
+		(property "Reference" "#PWR0250"
 			(at 194.31 102.87 0)
 			(effects
@@
 			(project "flight-core"
 				(path "/93f46f4b-cdf5-47ec-af03-96378e73b2e1/f120f04e-9926-485a-8729-a726a206f3dc"
-					(reference "#PWR0220")
+					(reference "#PWR0250")
 					(unit 1)
 				)
@@
 		(dnp no)
 		(fields_autoplaced yes)
-		(property "Reference" "#PWR0216"
+		(property "Reference" "#PWR0246"
 			(at 139.7 123.19 0)
 			(effects
@@
 			(project "flight-core"
 				(path "/93f46f4b-cdf5-47ec-af03-96378e73b2e1/f120f04e-9926-485a-8729-a726a206f3dc"
-					(reference "#PWR0216")
+					(reference "#PWR0246")
 					(unit 1)
 				)
@@
 		(dnp no)
 		(fields_autoplaced yes)
-		(property "Reference" "#PWR0223"
+		(property "Reference" "#PWR0253"
 			(at 241.3 139.7 0)
 			(effects
@@
 			(project "flight-core"
 				(path "/93f46f4b-cdf5-47ec-af03-96378e73b2e1/f120f04e-9926-485a-8729-a726a206f3dc"
-					(reference "#PWR0223")
+					(reference "#PWR0253")
 					(unit 1)
 				)
@@
 		(dnp no)
 		(fields_autoplaced yes)
-		(property "Reference" "U59"
+		(property "Reference" "U58"
 			(at 119.38 53.34 0)
 			(effects
@@
 			(project "flight-core"
 				(path "/93f46f4b-cdf5-47ec-af03-96378e73b2e1/f120f04e-9926-485a-8729-a726a206f3dc"
-					(reference "U59")
+					(reference "U58")
 					(unit 1)
 				)
@@
 		(dnp no)
 		(fields_autoplaced yes)
-		(property "Reference" "U57"
+		(property "Reference" "U56"
 			(at 82.55 115.57 0)
 			(effects
@@
 			(project ""
 				(path "/93f46f4b-cdf5-47ec-af03-96378e73b2e1/f120f04e-9926-485a-8729-a726a206f3dc"
-					(reference "U57")
+					(reference "U56")
 					(unit 1)
 				)
@@
 		(on_board yes)
 		(dnp no)
-		(property "Reference" "U58"
+		(property "Reference" "U57"
 			(at 104.775 113.03 0)
 			(effects
@@
 			(project "flight-core"
 				(path "/93f46f4b-cdf5-47ec-af03-96378e73b2e1/f120f04e-9926-485a-8729-a726a206f3dc"
-					(reference "U58")
+					(reference "U57")
 					(unit 1)
 				)
@@
 		(on_board yes)
 		(dnp no)
-		(property "Reference" "R50"
+		(property "Reference" "R64"
 			(at 47.498 46.482 90)
 			(effects
@@
 			(project ""
 				(path "/93f46f4b-cdf5-47ec-af03-96378e73b2e1/f120f04e-9926-485a-8729-a726a206f3dc"
-					(reference "R50")
+					(reference "R64")
 					(unit 1)
 				)
@@
 		(on_board yes)
 		(dnp no)
-		(property "Reference" "R53"
+		(property "Reference" "R67"
 			(at 71.628 73.152 90)
 			(effects
@@
 			(project ""
 				(path "/93f46f4b-cdf5-47ec-af03-96378e73b2e1/f120f04e-9926-485a-8729-a726a206f3dc"
-					(reference "R53")
+					(reference "R67")
 					(unit 1)
 				)
@@
 		(on_board yes)
 		(dnp no)
-		(property "Reference" "R51"
+		(property "Reference" "R65"
 			(at 46.99 59.69 90)
 			(effects
@@
 			(project ""
 				(path "/93f46f4b-cdf5-47ec-af03-96378e73b2e1/f120f04e-9926-485a-8729-a726a206f3dc"
-					(reference "R51")
+					(reference "R65")
 					(unit 1)
 				)
@@
 		(on_board yes)
 		(dnp no)
-		(property "Reference" "U62"
+		(property "Reference" "U61"
 			(at 207.645 113.665 0)
 			(effects
@@
 			(project "flight-core"
 				(path "/93f46f4b-cdf5-47ec-af03-96378e73b2e1/f120f04e-9926-485a-8729-a726a206f3dc"
-					(reference "U62")
+					(reference "U61")
 					(unit 1)
 				)
@@
 		(dnp no)
 		(fields_autoplaced yes)
-		(property "Reference" "#PWR0222"
+		(property "Reference" "#PWR0252"
 			(at 241.3 124.46 0)
 			(effects
@@
 			(project "flight-core"
 				(path "/93f46f4b-cdf5-47ec-af03-96378e73b2e1/f120f04e-9926-485a-8729-a726a206f3dc"
-					(reference "#PWR0222")
+					(reference "#PWR0252")
 					(unit 1)
 				)
@@
 		(dnp no)
 		(fields_autoplaced yes)
-		(property "Reference" "#PWR0213"
+		(property "Reference" "#PWR0243"
 			(at 73.66 81.28 0)
 			(effects
@@
 			(project "flight-core"
 				(path "/93f46f4b-cdf5-47ec-af03-96378e73b2e1/f120f04e-9926-485a-8729-a726a206f3dc"
-					(reference "#PWR0213")
+					(reference "#PWR0243")
 					(unit 1)
 				)
@@
 		(on_board yes)
 		(dnp no)
-		(property "Reference" "Q5"
+		(property "Reference" "Q20"
 			(at 75.184 58.674 90)
 			(effects
@@
 			(project "flight-core"
 				(path "/93f46f4b-cdf5-47ec-af03-96378e73b2e1/f120f04e-9926-485a-8729-a726a206f3dc"
-					(reference "Q5")
+					(reference "Q20")
 					(unit 1)
 				)
@@
 		(dnp no)
 		(fields_autoplaced yes)
-		(property "Reference" "U60"
+		(property "Reference" "U59"
 			(at 187.96 116.84 0)
 			(effects
@@
 			(project "flight-core"
 				(path "/93f46f4b-cdf5-47ec-af03-96378e73b2e1/f120f04e-9926-485a-8729-a726a206f3dc"
-					(reference "U60")
+					(reference "U59")
 					(unit 1)
 				)
@@
 		(dnp no)
 		(fields_autoplaced yes)
-		(property "Reference" "#PWR0212"
+		(property "Reference" "#PWR0242"
 			(at 60.96 81.28 0)
 			(effects
@@
 			(project "flight-core"
 				(path "/93f46f4b-cdf5-47ec-af03-96378e73b2e1/f120f04e-9926-485a-8729-a726a206f3dc"
-					(reference "#PWR0212")
+					(reference "#PWR0242")
 					(unit 1)
 				)
@@
 		(on_board yes)
 		(dnp no)
-		(property "Reference" "#PWR0218"
+		(property "Reference" "#PWR0248"
 			(at 147.32 81.28 0)
 			(effects
@@
 			(project "flight-core"
 				(path "/93f46f4b-cdf5-47ec-af03-96378e73b2e1/f120f04e-9926-485a-8729-a726a206f3dc"
-					(reference "#PWR0218")
+					(reference "#PWR0248")
 					(unit 1)
 				)
@@
 		(dnp no)
 		(fields_autoplaced yes)
-		(property "Reference" "U61"
+		(property "Reference" "U60"
 			(at 194.31 52.07 0)
 			(effects
@@
 			(project "flight-core"
 				(path "/93f46f4b-cdf5-47ec-af03-96378e73b2e1/f120f04e-9926-485a-8729-a726a206f3dc"
-					(reference "U61")
+					(reference "U60")
 					(unit 1)
 				)
@@
 		(dnp no)
 		(fields_autoplaced yes)
-		(property "Reference" "#PWR0219"
+		(property "Reference" "#PWR0249"
 			(at 168.91 58.42 0)
 			(effects
@@
 			(project ""
 				(path "/93f46f4b-cdf5-47ec-af03-96378e73b2e1/f120f04e-9926-485a-8729-a726a206f3dc"
-					(reference "#PWR0219")
+					(reference "#PWR0249")
 					(unit 1)
 				)
@@
 		(on_board yes)
 		(dnp no)
-		(property "Reference" "D7"
+		(property "Reference" "D22"
 			(at 44.45 64.262 0)
 			(effects
@@
 			(project ""
 				(path "/93f46f4b-cdf5-47ec-af03-96378e73b2e1/f120f04e-9926-485a-8729-a726a206f3dc"
-					(reference "D7")
+					(reference "D22")
 					(unit 1)
 				)
@@
 		(on_board yes)
 		(dnp no)
-		(property "Reference" "R52"
+		(property "Reference" "R66"
 			(at 57.912 64.262 90)
 			(effects
@@
 			(project "flight-core"
 				(path "/93f46f4b-cdf5-47ec-af03-96378e73b2e1/f120f04e-9926-485a-8729-a726a206f3dc"
-					(reference "R52")
+					(reference "R66")
 					(unit 1)
 				)
@@
 		(dnp no)
 		(fields_autoplaced yes)
-		(property "Reference" "#PWR0217"
+		(property "Reference" "#PWR0247"
 			(at 139.7 138.43 0)
 			(effects
@@
 			(project "flight-core"
 				(path "/93f46f4b-cdf5-47ec-af03-96378e73b2e1/f120f04e-9926-485a-8729-a726a206f3dc"
-					(reference "#PWR0217")
+					(reference "#PWR0247")
 					(unit 1)
 				)
@@
 		(dnp no)
 		(fields_autoplaced yes)
-		(property "Reference" "#PWR0221"
+		(property "Reference" "#PWR0251"
 			(at 223.52 139.7 0)
 			(effects
@@
 			(project "flight-core"
 				(path "/93f46f4b-cdf5-47ec-af03-96378e73b2e1/f120f04e-9926-485a-8729-a726a206f3dc"
-					(reference "#PWR0221")
+					(reference "#PWR0251")
 					(unit 1)
 				)
@@
 		(on_board yes)
 		(dnp no)
-		(property "Reference" "#PWR0214"
+		(property "Reference" "#PWR0244"
 			(at 93.98 81.28 0)
 			(effects
@@
 			(project "flight-core"
 				(path "/93f46f4b-cdf5-47ec-af03-96378e73b2e1/f120f04e-9926-485a-8729-a726a206f3dc"
-					(reference "#PWR0214")
+					(reference "#PWR0244")
 					(unit 1)
 				)
@@
 		(dnp no)
 		(fields_autoplaced yes)
-		(property "Reference" "#PWR0215"
+		(property "Reference" "#PWR0245"
 			(at 120.65 138.43 0)
 			(effects
@@
 			(project "flight-core"
 				(path "/93f46f4b-cdf5-47ec-af03-96378e73b2e1/f120f04e-9926-485a-8729-a726a206f3dc"
-					(reference "#PWR0215")
-					(unit 1)
-				)
+					(reference "#PWR0245")
+					(unit 1)
+				)
