File: Hardware/Core/flight-core/test_points_leds.kicad_sch (KiCad schematic)
At the start: 106 parts, among them Q10 MMBF170, Q11 MMBF170, Q12 MMBF170, Q13 MMBF170, Q14 MMBF170, Q15 MMBF170, Q16 MMBF170, Q17 MMBF170, Q18 MMBF170, Q19 MMBF170, Q20 MMBF170, Q21 MMBF170, Q22 MMBF170, Q23 MMBF170, Q24 MMBF170, Q25 MMBF170, Q26 MMBF170, Q27 MMBF170, Q28 MMBF170, Q29 MMBF170, Q9 MMBF170

Commit message: major component area placement begun, installing place footprints plugin, updating connectors to vertical
Parts:
- removed D16, D17, D19, D20, D22, D23, D24, D25, D26, D27, D28, D29, D30, D31, D32, D33, D34, D35, D36, D37, D38: LED_0805_Amber, footprints:LED_0805_OEM, symbol formula:LED_0805_Amber
- removed Q10, Q11, Q12, Q13, Q14, Q15, Q16, Q17, Q18, Q19, Q20, Q21, Q22, Q23, Q24, Q25, Q26, Q27, Q28, Q29, Q9: MMBF170, Package_TO_SOT_SMD:SOT-23, symbol formula:MMBF170
- removed R63, R65, R67, R68, R70, R71, R72, R73, R74, R75, R76, R77, R78, R79, R80, R81, R82, R83, R84, R85, R86: R_200, footprints:R_0603_1608Metric, symbol formula:R_200
- removed TP15, TP17, TP18, TP19, TP20, TP21, TP22, TP24, TP25, TP28, TP29, TP30, TP31, TP32, TP33, TP34, TP35, TP36, TP37, TP38, TP39: TP, footprints:tp_1.6mm, symbol formula:TP
- renumbered D11 to D25, D10 to D26, D13 to D27, D12 to D28, D14 to D29, D15 to D30, D18 to D31, D21 to D32, R59 to R72, R58 to R73, R61 to R74, R60 to R75, R62 to R76, R64 to R77, R66 to R78, R69 to R79, TP23 to TP30, TP16 to TP31, TP27 to TP32, TP26 to TP33
Connections:
- net SHDN_SENSE_RIDER_ESTOP renamed SHDN_SENSE_CRIT_RIDER_ESTOP
Other:
- added sheet shutdown LED circuit (shdn_led.kicad_sch)
- added sheet shutdown LED circuit1 (shdn_led.kicad_sch)
- added sheet shutdown LED circuit10 (shdn_led.kicad_sch)
- added sheet shutdown LED circuit11 (shdn_led.kicad_sch)
- added sheet shutdown LED circuit12 (shdn_led.kicad_sch)
- added sheet shutdown LED circuit13 (shdn_led.kicad_sch)
- added sheet shutdown LED circuit14 (shdn_led.kicad_sch)
- added sheet shutdown LED circuit15 (shdn_led.kicad_sch)
- added sheet shutdown LED circuit16 (shdn_led.kicad_sch)
- added sheet shutdown LED circuit17 (shdn_led.kicad_sch)
- added sheet shutdown LED circuit18 (shdn_led.kicad_sch)
- added sheet shutdown LED circuit19 (shdn_led.kicad_sch)
- added sheet shutdown LED circuit20 (shdn_led.kicad_sch)
- added sheet shutdown LED circuit21 (shdn_led.kicad_sch)
- added sheet shutdown LED circuit3 (shdn_led.kicad_sch)
- added sheet shutdown LED circuit4 (shdn_led.kicad_sch)
- added sheet shutdown LED circuit5 (shdn_led.kicad_sch)
- added sheet shutdown LED circuit6 (shdn_led.kicad_sch)
- added sheet shutdown LED circuit7 (shdn_led.kicad_sch)
- added sheet shutdown LED circuit8 (shdn_led.kicad_sch)
- added sheet shutdown LED circuit9 (shdn_led.kicad_sch)
- moved on the sheet: D25, D26, D27, D28, D29, D30, D31, D32, R72, R73, R74, R75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

Commit message: switching test points to correct footprint and alternative symbol, moving leds
Parts:
- TP_STM_IO1, TP_STM_IO2: footprint footprints:tp_1.6mm -> TestPoint:TestPoint_Pad_D1.0mm; symbol formula:TP -> OlinBAD:D1.0_TP
Other:
- moved on the sheet: TP_STM_IO1, TP_STM_IO2
Changed lines of the file:
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@@
 	)
 	(symbol
-		(lib_id "formula:TP")
-		(at 40.64 162.56 270)
-		(mirror x)
+		(lib_id "OlinBAD:D1.0_TP")
+		(at 35.56 162.56 0)
+		(mirror y)
 		(unit 1)
 		(exclude_from_sim no)
@@
 		(dnp no)
 		(property "Reference" "TP_STM_IO1"
-			(at 43.18 158.75 90)
+			(at 27.94 161.29 0)
 			(effects
 				(font
@@
 		)
 		(property "Value" "TP"
-			(at 43.18 161.29 90)
-			(effects
-				(font
-					(size 1.27 1.27)
-				)
-			)
-		)
-		(property "Footprint" "footprints:tp_1.6mm"
-			(at 38.1 165.1 0)
-			(effects
-				(font
-					(size 1.27 1.27)
-				)
-				(hide yes)
-			)
-		)
-		(property "Datasheet" "http://www.keyelco.com/product-pdf.cfm?p=1314"
-			(at 40.64 162.56 0)
-			(effects
-				(font
-					(size 1.27 1.27)
-				)
-				(hide yes)
-			)
-		)
-		(property "Description" ""
-			(at 40.64 162.56 0)
+			(at 27.94 158.75 0)
+			(effects
+				(font
+					(size 1.27 1.27)
+				)
+			)
+		)
+		(property "Footprint" "TestPoint:TestPoint_Pad_D1.0mm"
+			(at 30.48 162.56 0)
+			(effects
+				(font
+					(size 1.27 1.27)
+				)
+				(hide yes)
+			)
+		)
+		(property "Datasheet" "~"
+			(at 30.48 162.56 0)
+			(effects
+				(font
+					(size 1.27 1.27)
+				)
+				(hide yes)
+			)
+		)
+		(property "Description" "test point"
+			(at 35.56 162.56 0)
 			(effects
 				(font
@@
 		)
 		(property "MFN" "DK"
-			(at 43.18 160.02 0)
+			(at 33.02 160.02 0)
 			(effects
 				(font
@@
 		)
 		(property "MPN" "36-5006-ND"
-			(at 45.72 157.48 0)
+			(at 30.48 157.48 0)
 			(effects
 				(font
@@
 		)
 		(property "PurchasingLink" "https://www.digikey.com/product-detail/en/keystone-electronics/5006/36-5006-ND/255330"
-			(at 48.26 154.94 0)
+			(at 27.94 154.94 0)
 			(effects
 				(font
@@
 	)
 	(symbol
-		(lib_id "formula:TP")
-		(at 71.12 162.56 270)
-		(mirror x)
+		(lib_id "OlinBAD:D1.0_TP")
+		(at 66.04 162.56 0)
+		(mirror y)
 		(unit 1)
 		(exclude_from_sim no)
@@
 		(dnp no)
 		(property "Reference" "TP_STM_IO2"
-			(at 73.66 158.75 90)
+			(at 58.42 161.29 0)
 			(effects
 				(font
@@
 		)
 		(property "Value" "TP"
-			(at 73.66 161.29 90)
-			(effects
-				(font
-					(size 1.27 1.27)
-				)
-			)
-		)
-		(property "Footprint" "footprints:tp_1.6mm"
-			(at 68.58 165.1 0)
-			(effects
-				(font
-					(size 1.27 1.27)
-				)
-				(hide yes)
-			)
-		)
-		(property "Datasheet" "http://www.keyelco.com/product-pdf.cfm?p=1314"
-			(at 71.12 162.56 0)
-			(effects
-				(font
-					(size 1.27 1.27)
-				)
-				(hide yes)
-			)
-		)
-		(property "Description" ""
-			(at 71.12 162.56 0)
+			(at 58.42 158.75 0)
+			(effects
+				(font
+					(size 1.27 1.27)
+				)
+			)
+		)
+		(property "Footprint" "TestPoint:TestPoint_Pad_D1.0mm"
+			(at 60.96 162.56 0)
+			(effects
+				(font
+					(size 1.27 1.27)
+				)
+				(hide yes)
+			)
+		)
+		(property "Datasheet" "~"
+			(at 60.96 162.56 0)
+			(effects
+				(font
+					(size 1.27 1.27)
+				)
+				(hide yes)
+			)
+		)
+		(property "Description" "test point"
+			(at 66.04 162.56 0)
 			(effects
 				(font
@@
 		)
 		(property "MFN" "DK"
-			(at 73.66 160.02 0)
+			(at 63.5 160.02 0)
 			(effects
 				(font
@@
 		)
 		(property "MPN" "36-5006-ND"
-			(at 76.2 157.48 0)
+			(at 60.96 157.48 0)
 			(effects
 				(font
@@
 		)
 		(property "PurchasingLink" "https://www.digikey.com/product-detail/en/keystone-electronics/5006/36-5006-ND/255330"
-			(at 78.74 154.94 0)
-			(effects
-				(font
+			(at 58.42 154.94 0)
+			(effects
+				(font

Commit message: updating mini tps to new symbol and footprint
Parts:
- TP_STM_IO1, TP_STM_IO2: footprint TestPoint:TestPoint_Pad_D1.0mm -> obad_footprints:TestPoint_Pad_D1.0mm
Changed lines of the file:
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@@
 			)
 		)
-		(property "Footprint" "TestPoint:TestPoint_Pad_D1.0mm"
+		(property "Footprint" "obad_footprints:TestPoint_Pad_D1.0mm"
 			(at 30.48 162.56 0)
 			(effects
@@
 			)
 		)
-		(property "Footprint" "TestPoint:TestPoint_Pad_D1.0mm"
+		(property "Footprint" "obad_footprints:TestPoint_Pad_D1.0mm"
 			(at 60.96 162.56 0)
 			(effects
