File: Hardware/Core/flight-core/shdn.kicad_sch (KiCad schematic)
At the start: 23 parts, among them J14 Conn_02x02_Remote_ESTOP, J15 Conn_02x07_Counter_Clockwise, J16 Conn_02x02_Remote_ESTOP, J19 Conn_02x02_Remote_ESTOP, J20 Conn_02x02_Remote_ESTOP, J21 Conn_02x02_Remote_ESTOP, J22 Conn_02x02_Remote_ESTOP, J23 Conn_02x02_Remote_ESTOP, J24 Conn_02x02_Remote_ESTOP, J25 Conn_02x02_Remote_ESTOP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

Commit message: minor reformatting; no substantial changes
Parts:
- J3201: value Conn_02x02_Remote_ESTOP -> Conn_02x02_TILT
Changed lines of the file:
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@@
 			)
 		)
-		(property "Value" "Conn_02x02_Remote_ESTOP"
+		(property "Value" "Conn_02x02_TILT"
 			(at 49.53 46.99 0)
 			(effects
