File: Hardware/Core/flight-core/shdn_no_tp.kicad_sch (KiCad schematic)
At the start: 3 parts, among them Q5 MMBF170

Commit message: minor reformatting; no substantial changes
Other:
- note added: "Forgot a 100k pull-down attached to the SHDNs! Will be soldering these on by hand..."
Changed lines of the file:
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@@
 	(generator_version "9.0")
 	(paper "A5")
+	(text "Forgot a 100k pull-down attached to the SHDNs! \nWill be soldering these on by hand..."
+		(exclude_from_sim no)
+		(at 80.01 79.375 0)
+		(effects
+			(font
+				(size 1.27 1.27)
+			)
+		)
+	)
 	(wire
 		(pts
