File: Hardware/Charger/Charger/converters.kicad_sch (KiCad schematic)
At the start: 38 parts, among them J201 Conn_01x02, U202 Fuse_Holder_Blade, U204 Fuse_Holder_Blade

Commit message: built charger schematic and added parts to layout
Parts:
- removed U202, U204: Fuse_Holder_Blade, footprints:Fuse_Block_Holder, symbol formula:Fuse_Holder_Blade
- added F201, F202: Fuse 1A, Fuse:Fuse_1206_3216Metric, symbol Device:Fuse
- gave numbers to parts that had none: 14
- renumbered C201 to C202, C202 to C204, C203 to C206, C204 to C208, C205 to C210, C206 to C212, C207 to C214, C208 to C216, C209 to C218, D101 to D204, D102 to D205, L201 to L202, R201 to R202, R202 to R205, R203 to R206, R101 to R207, R102 to R208, U201 to U202
Connections:
- net +3.3V: now also F202.2
- net +5V: now also F201.1
- net at C208.1, C212.1, C214.1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: now also F202.1
- net at C207.1, C211.1, C213.1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: now also F201.2

Commit message: Few updates to connectors
Connections:
- net +12V renamed +24V
Other:
- note added: "Connector to +24V Supply"
- note removed: "Connector to +12V Supply"
Changed lines of the file:
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@@
 		)
 	)
-	(text "Connector to +12V Supply"
+	(text "Connector to +24V Supply"
 		(exclude_from_sim no)
 		(at 78.232 86.614 0)
@@
 		)
 	)
-	(hierarchical_label "+12V"
-		(shape input)
-		(at 83.82 96.52 0)
-		(effects
-			(font
-				(size 1.27 1.27)
-			)
-			(justify left)
-		)
-	)
 	(hierarchical_label "3.3V"
 		(shape output)
@@
 		)
 	)
-	(hierarchical_label "+12V"
-		(shape input)
-		(at 110.49 110.49 180)
-		(effects
-			(font
-				(size 1.27 1.27)
-			)
-			(justify right)
-		)
-	)
 	(hierarchical_label "5v_USBC"
 		(shape input)
@@
 		(shape input)
 		(at 214.63 125.73 180)
-		(effects
-			(font
-				(size 1.27 1.27)
-			)
-			(justify right)
-		)
-	)
-	(hierarchical_label "+12V"
-		(shape input)
-		(at 102.87 43.18 180)
 		(effects
 			(font
@@
 	)
 	(symbol
+		(lib_id "power:+24V")
+		(at 102.87 43.18 0)
+		(unit 1)
+		(exclude_from_sim no)
+		(in_bom yes)
+		(on_board yes)
+		(dnp no)
+		(fields_autoplaced yes)
+		(property "Reference" "#PWR0214"
+			(at 102.87 46.99 0)
+			(effects
+				(font
+					(size 1.27 1.27)
+				)
+				(hide yes)
+			)
+		)
+		(property "Value" "+24V"
+			(at 102.87 38.1 0)
+			(effects
+				(font
+					(size 1.27 1.27)
+				)
+			)
+		)
+		(property "Footprint" ""
+			(at 102.87 43.18 0)
+			(effects
+				(font
+					(size 1.27 1.27)
+				)
+				(hide yes)
+			)
+		)
+		(property "Datasheet" ""
+			(at 102.87 43.18 0)
+			(effects
+				(font
+					(size 1.27 1.27)
+				)
+				(hide yes)
+			)
+		)
+		(property "Description" "Power symbol creates a global label with name \"+24V\""
+			(at 102.87 43.18 0)
+			(effects
+				(font
+					(size 1.27 1.27)
+				)
+				(hide yes)
+			)
+		)
+		(pin "1"
+		)
+		(instances
+			(project "Charger"
+				(path "/ec0cb266-3da5-4155-a0e5-38a3c68d3210/91227ca9-06bc-4f19-ad47-eac0cfdbbcc1"
+					(reference "#PWR0214")
+					(unit 1)
+				)
+			)
+		)
+	)
+	(symbol
+		(lib_id "power:+24V")
+		(at 110.49 110.49 0)
+		(unit 1)
+		(exclude_from_sim no)
+		(in_bom yes)
+		(on_board yes)
+		(dnp no)
+		(fields_autoplaced yes)
+		(property "Reference" "#PWR0213"
+			(at 110.49 114.3 0)
+			(effects
+				(font
+					(size 1.27 1.27)
+				)
+				(hide yes)
+			)
+		)
+		(property "Value" "+24V"
+			(at 110.49 105.41 0)
+			(effects
+				(font
+					(size 1.27 1.27)
+				)
+			)
+		)
+		(property "Footprint" ""
+			(at 110.49 110.49 0)
+			(effects
+				(font
+					(size 1.27 1.27)
+				)
+				(hide yes)
+			)
+		)
+		(property "Datasheet" ""
+			(at 110.49 110.49 0)
+			(effects
+				(font
+					(size 1.27 1.27)
+				)
+				(hide yes)
+			)
+		)
+		(property "Description" "Power symbol creates a global label with name \"+24V\""
+			(at 110.49 110.49 0)
+			(effects
+				(font
+					(size 1.27 1.27)
+				)
+				(hide yes)
+			)
+		)
+		(pin "1"
+		)
+		(instances
+			(project "Charger"
+				(path "/ec0cb266-3da5-4155-a0e5-38a3c68d3210/91227ca9-06bc-4f19-ad47-eac0cfdbbcc1"
+					(reference "#PWR0213")
+					(unit 1)
+				)
+			)
+		)
+	)
+	(symbol
 		(lib_id "Device:C")
 		(at 173.99 68.58 0)
@@
 					(unit 1)
 				)
+			)
+		)
+	)
+	(symbol
+		(lib_id "power:+24V")
+		(at 83.82 96.52 0)
+		(unit 1)
+		(exclude_from_sim no)
+		(in_bom yes)
+		(on_board yes)
+		(dnp no)
+		(fields_autoplaced yes)
+		(property "Reference" "#PWR0212"
+			(at 83.82 100.33 0)
+			(effects
+				(font
+					(size 1.27 1.27)
+				)
+				(hide yes)
+			)
+		)
+		(property "Value" "+24V"
+			(at 83.82 91.44 0)
+			(effects
+				(font
+					(size 1.27 1.27)
+				)
+			)
+		)
+		(property "Footprint" ""
+			(at 83.82 96.52 0)
+			(effects
+				(font
+					(size 1.27 1.27)
+				)
+				(hide yes)
+			)
+		)
+		(property "Datasheet" ""
+			(at 83.82 96.52 0)
+			(effects
+				(font
+					(size 1.27 1.27)
+				)
+				(hide yes)
+			)
+		)
+		(property "Description" "Power symbol creates a global label with name \"+24V\""
+			(at 83.82 96.52 0)
+			(effects
+				(font
+					(size 1.27 1.27)
+				)
+				(hide yes)
+			)
+		)
+		(pin "1"
+		)
+		(instances
+			(project ""
+				(path "/ec0cb266-3da5-4155-a0e5-38a3c68d3210/91227ca9-06bc-4f19-ad47-eac0cfdbbcc1"
+					(reference "#PWR0212")
+					(unit 1)
+				)

Commit message: Completed PCB layout of charger
Parts:
- renumbered C209 to C10, C210 to C11, C211 to C12, C212 to C13, C213 to C14, C214 to C15, C215 to C16, C216 to C17, C217 to C18, C218 to C19, C201 to C2, C202 to C3, C203 to C4, C204 to C5, C205 to C6, C206 to C7, C207 to C8, C208 to C9, D201 to D3, D202 to D4, D203 to D5, D204 to D6, D205 to D7, F201 to F1, F202 to F2, J201 to J4, L201 to L1, L202 to L2, R201 to R11, R202 to R12, R203 to R13, R204 to R14, R205 to R15, R206 to R16, R207 to R17, R208 to R18, U201 to U1, U202 to U2
