File: Hardware/Cube-Flipper/flipper/flipper.kicad_pcb (KiCad board)
At the start: 2 copper layers, 38.2 x 38.2 mm, 3 parts, among them J1 Cube Orange Plus Male Header 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, J2 Cube Orange Plus Female Header

Commit message: routing most of it
Routing:
- net /CAN+: track 0.00 -> 59.9 mm, vias 0 -> 1
- net /CAN-: track 0.00 -> 56.9 mm, vias 0 -> 1
- net /SBUS_IO_B: track 0.00 -> 49.7 mm, vias 0 -> 3
- net /SBUS_IO_A: track 0.00 -> 47.8 mm, vias 0 -> 3
- net /TP_P60: track 0.00 -> 45.5 mm, vias 0 -> 3
- net /TP_P58: track 0.00 -> 43.2 mm, vias 0 -> 3
- net /UART_TELEM1_RX: track 0.00 -> 41.1 mm, vias 0 -> 1
- net /TP_P56: track 0.00 -> 41.0 mm, vias 0 -> 3
- net /UART_TELEM1_TX: track 0.00 -> 40.2 mm, vias 0 -> 1
- net /UART_TELEM1_RTS: track 0.00 -> 38.3 mm, vias 0 -> 1
- net /CUBE_HANDOFF: track 0.00 -> 38.2 mm, vias 0 -> 3
- net /UART_TELEM1_CTS: track 0.00 -> 37.0 mm, vias 0 -> 1
- net /FMU_LED_AMBER: track 0.00 -> 32.5 mm, vias 0 -> 1
- net /+5V: track 0.00 -> 29.9 mm, vias 0 -> 1
- net /IO_~{RESET}: track 0.00 -> 28.7 mm, vias 0 -> 1
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
Commit message: complete flipper i really hope I didn't cook it
Parts:
- removed REF**: CONN_DF173p0H-80DS-0p5V57_80P_HIR, obad_footprints:CONN_DF173p0H-80DS-0p5V57_80P_HIR
Connections:
- J1 pad 30: /UART_TELEM2_RX -> unconnected-(J1-Pad30)
- J1 pad 32: /UART_TELEM2_TX -> unconnected-(J1-Pad32)
- J1 pad 34: /UART_TELEM2_RTS -> unconnected-(J1-Pad34)
- J1 pad 36: /UART_TELEM2_CTS -> unconnected-(J1-Pad36)
- J2 pad 30: /UART_TELEM2_RX -> unconnected-(J2-Pad30)
- J2 pad 32: /UART_TELEM2_TX -> unconnected-(J2-Pad32)
- J2 pad 34: /UART_TELEM2_RTS -> unconnected-(J2-Pad34)
- J2 pad 36: /UART_TELEM2_CTS -> unconnected-(J2-Pad36)
Routing:
- net /SHDN_CRITICAL: track 0.00 -> 9.08 mm, vias 0 -> 1
- net /GND: track 0.00 -> 6.30 mm, vias 0 -> 124
- net /+5V: track 29.9 -> 35.2 mm
- net /CAN+: track 59.9 -> 56.2 mm
- net /CAN-: track 56.9 -> 53.8 mm, vias 1 -> 3
- net /FINAL_SHDN: track 8.43 -> 11.1 mm
- net /TP_P56: track 41.0 -> 42.7 mm
- net /TP_P58: track 43.2 -> 44.5 mm
- net /TP_P60: track 45.5 -> 46.6 mm
- net /SBUS_IO_B: track 49.7 -> 50.8 mm
- net /SBUS_IO_A: track 47.8 -> 48.8 mm
- net /ALARM: track 13.0 -> 13.8 mm
- net /CUBE_HANDOFF: track 38.2 -> 38.8 mm
- net /IO_SWCLK: track 27.3 -> 27.9 mm
- net /IO_SWDIO: track 25.9 -> 26.4 mm
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- added copper zone on B.Cu, net /GND
- added copper zone on F.Cu, net /GND
